File: Impression5-SMASH-Shield.brd (EAGLE design)
At the start: 115.6 x 74.9 mm, 113 parts, among them IC1 7805TV, J1 1725656, J10 61300811121, J11 61300811121, J12 61300611121, J13 61300311121, J14 61300311121, J15 61300311121, J16 61300311121, J17 61300311121, J18 61300311121, J19 61300611121, J2 1725656, J20 61300311121, J21 61300311121, J22 61300411121, J23 61300311121, J24 61300311121, J25 61300311121, J26 61300311121, J27 61300311121, J28 61300311121, J29 61300311121, J3 1725656, J30 61300311121, J31 61300311121, J32 61300311121, J33 61300311121, J34 61300311121, J35 61300311121, J36 61300311121, J37 61300311121, J38 61300311121, J39 61300311121, J4 1725656, J40 61300311121, J41 61300311121, J42 61300311121, J43 61300211121, J44 61300211121, J45 61300211121, J46 61300211121, J47 61300811121, J48 61300311121, J49 61300311121, J5 1725656, J50 61300311121, J51 61300311121, J52 61300611121, J53 61300811121, J54 61300811121, J6 1725656, J7 1725656, J8 1725656, J9 1725656, Q1 IRF512, Q2 IRF512, Q3 IRF512, Q4 IRF512, Q5 IRF512, Q6 IRF512, Q7 IRF512, Q8 IRF512

Commit message: changed 4/2V to 5VL. This powers the VDD of the TLC5917 and needs to be 5V.
Parts:
- R17, R19: value 10k -> 243
- R18: value 10k -> 729R
Connections:
- net 4/2V renamed 5VL
Changed lines of the file:
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@@
 <attribute name="NAME" x="76.2" y="33.02" size="1.016" layer="25"/>
 </element>
-<element name="R17" library="SparkFun" package="AXIAL-0.3" value="10k" x="71.12" y="31.115" smashed="yes">
+<element name="R17" library="SparkFun" package="AXIAL-0.3" value="243" x="71.12" y="31.115" smashed="yes">
 <attribute name="NAME" x="76.073" y="30.607" size="1.016" layer="25"/>
 </element>
@@
 <attribute name="VALUE" x="76.2" y="22.86" size="1.27" layer="27" ratio="10" rot="R180"/>
 </element>
-<element name="R18" library="SparkFun" package="AXIAL-0.3" value="10k" x="71.12" y="23.495" smashed="yes">
+<element name="R18" library="SparkFun" package="AXIAL-0.3" value="729R" x="71.12" y="23.495" smashed="yes">
 <attribute name="NAME" x="76.2" y="23.495" size="1.016" layer="25"/>
 </element>
-<element name="R19" library="SparkFun" package="AXIAL-0.3" value="10k" x="71.12" y="20.955" smashed="yes">
+<element name="R19" library="SparkFun" package="AXIAL-0.3" value="243" x="71.12" y="20.955" smashed="yes">
 <attribute name="NAME" x="76.835" y="20.32" size="1.016" layer="25"/>
 </element>
@@
 <wire x1="71.12" y1="26.035" x2="71.12" y2="27.94" width="1.27" layer="1"/>
 </signal>
-<signal name="4/2V">
+<signal name="5VL">
 <contactref element="J47" pad="1"/>
 <contactref element="R19" pad="P$1"/>

Commit message: Changed the 8/5V to 9/5V, actually 9V2 and 5V0 respectively. These voltages needs to provide the maximum Vf that the 7-Segments may need. The max Vf are: SA23-11SRWA = 9.2V SA15-11EWA  = 5.0V
Parts:
- R16: value 10k -> 1551R or 729R
Connections:
- net 8/5V renamed 9/5V
Changed lines of the file:
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@@
 <attribute name="VALUE" x="76.2" y="33.02" size="1.27" layer="27" ratio="10" rot="R180"/>
 </element>
-<element name="R16" library="SparkFun" package="AXIAL-0.3" value="10k" x="71.12" y="33.655" smashed="yes">
+<element name="R16" library="SparkFun" package="AXIAL-0.3" value="1551R or 729R" x="71.12" y="33.655" smashed="yes">
 <attribute name="NAME" x="76.2" y="33.02" size="1.016" layer="25"/>
 </element>
@@
 <via x="19.05" y="50.8" extent="1-16" drill="1.1" diameter="1.8796"/>
 </signal>
-<signal name="8/5V">
+<signal name="9/5V">
 <contactref element="J47" pad="7"/>
 <contactref element="R17" pad="P$1"/>
